File: eagle/v1.brd (EAGLE design)
At the start: 24.2 x 49.6 mm, 48 parts, among them IC2 LT1761, IC4 LT1376-ADJ, Q1 12Mhz, T1 Si2301DS, X1 USB-MICROB

Commit message: turned usb
Parts:
- moved T1 8.69 mm to (16.4, -11.1)
- moved R9 8.26 mm to (16.1, -14.1), turned to 0 degrees
- moved X1 5.62 mm to (25.3, -10.1), turned to 90 degrees
- moved R8 5.25 mm to (20.1, -13.5)
- moved R2 5.12 mm to (21.4, -13.5)
- moved R4 3.47 mm to (20.2, -11.1), turned to 0 degrees
- moved R12 3.40 mm to (15.6, -7.00), turned to 0 degrees
- moved R5 2.35 mm to (20.2, -9.78), turned to 0 degrees
- moved R13 1.79 mm to (15.6, -5.60), turned to 0 degrees
- moved BL 1.40 mm to (5.46, 1.50)
- moved C6 1.00 mm to (12.4, -6.80)
- moved 5V 0.80 mm to (13.2, -12.2)
- moved IC2 0.80 mm to (9.60, -6.80)
- moved SCK 0.80 mm to (10.2, -12.2)
- moved GND1 0.80 mm to (4.20, -12.2)
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Routing:
- net N$2: track 4.35 -> 16.8 mm, vias 0 -> 2
- net VBUS: track 9.10 -> 16.4 mm, vias 0 -> 2
- net N$14: track 4.09 -> 9.67 mm
- net GND: track 25.2 -> 20.4 mm, vias 31 -> 34
- net 06: track 7.14 -> 10.7 mm, vias 0 -> 2
- net SDA: track 37.1 -> 40.3 mm
- net N$24: track 4.41 -> 7.36 mm
- net N$8: track 38.8 -> 41.5 mm
- net +3V3: track 73.0 -> 70.8 mm, vias 4 -> 3
- net +5V: track 85.4 -> 83.8 mm
- net +5V_USB: track 2.43 -> 3.91 mm
- net N$11: track 3.12 -> 2.06 mm
- net 01: track 15.3 -> 14.6 mm
- net SCL: track 35.5 -> 36.1 mm

Commit message: refinements
Parts:
- moved R2 1.40 mm to (20.2, -12.7), turned to 180 degrees
- moved R8 0.82 mm to (20.2, -14.3), turned to 180 degrees
- moved R9 0.43 mm to (16.5, -14.0), turned to 180 degrees
- moved R7 0.30 mm to (7.70, 23.8)
- moved C4 0.20 mm to (19.3, 7.24)
- moved C5 0.20 mm to (12.8, 0.09)
- moved T1 0.20 mm to (16.6, -11.1)
- moved C6 0.15 mm to (12.6, -6.80)
- moved R4 0.10 mm to (20.2, -11.2)
- moved R5 0.10 mm to (20.2, -9.68)
Connections:
- net N$8: now also IC1.39
Routing:
- net N$2: track 16.8 -> 13.5 mm
- net +5V_USB: track 3.91 -> 3.05 mm
- net ADC: track 43.3 -> 43.8 mm
- net N$8: track 41.5 -> 42.0 mm
- net GND: track 20.4 -> 20.0 mm, vias 34 -> 33
